Commit message: rename dynaarm_end_effectors to duatic_dynaarm_end_effectors

File: duatic_dynaarm_end_effectors/urdf/freedrive_handle.urdf.xacro (robot description, xacro)
@@ -21,16 +21,16 @@
 THE USE OF THIS SOFTWARE, EVEN IF ADVISED OF THE POSSIBILITY OF SUCH DAMAGE.
 -->
-<robot name="weight_5kg" xmlns:xacro="http://www.ros.org/wiki/xacro">
+<robot name="freedrive_handle" xmlns:xacro="http://www.ros.org/wiki/xacro">
   <!-- Link Definition -->
-<xacro:macro name="weight_5kg" params="tf_prefix parent *origin">
-  <link name="${tf_prefix}weight_5kg_link">
+<xacro:macro name="freedrive_handle" params="tf_prefix parent *origin">
+  <link name="${tf_prefix}freedrive_handle_link">
     <!-- Inertial Properties -->
     <inertial>
-      <origin xyz="0.026295 0 0.000104" rpy="0 0 0"/>
-      <mass value="5.417999"/>
+      <origin xyz="0.0423 0 0" rpy="0 0 0"/>
+      <mass value="0.149"/>
       <inertia
-        ixx="0.031114" ixy="0.0"  ixz="0.000015"
-        iyy="0.015956" iyz="0.0"
-        izz=" 0.019591"/>
+        ixx=" 0.0000520" ixy="0.0"  ixz="0.0"
+        iyy="0.0001585" iyz="0.0"
+        izz="0.0001585"/>
     </inertial>
     <!-- Visual -->
@@ -38,5 +38,5 @@
       <origin xyz="0 0 0" rpy="0 0 0"/>
       <geometry>
-      <mesh filename="file://$(find dynaarm_end_effectors)/meshes/weight_mesh.stl" scale="1 1 1"/>
+      <mesh filename="file://$(find duatic_dynaarm_end_effectors)/meshes/freedrive_handle_mesh.stl" scale="1 1 1"/>
       </geometry>
       <material name="gray">
@@ -47,12 +47,12 @@
       <origin xyz="0 0 0" rpy="0 0 0"/>
       <geometry>
-      <mesh filename="file://$(find dynaarm_end_effectors)/meshes/weight_mesh.stl" scale="1 1 1"/>
+      <mesh filename="file://$(find duatic_dynaarm_end_effectors)/meshes/freedrive_handle_mesh.stl" scale="1 1 1"/>
       </geometry>
     </collision>
   </link>
   <!-- Fixed Joint to parent link -->
-  <joint name="${tf_prefix}weight_5kg_joint" type="fixed">
+  <joint name="${tf_prefix}freedrive_handle_joint" type="fixed">
     <parent link="${parent}"/>
-    <child link="${tf_prefix}weight_5kg_link"/>
+    <child link="${tf_prefix}freedrive_handle_link"/>
     <xacro:insert_block name="origin" />
   </joint>

File: duatic_dynaarm_end_effectors/urdf/freedrive_handle_standalone.urdf.xacro (robot description, xacro)
@@ -1,10 +1,10 @@
 <robot name="weight_on_world" xmlns:xacro="http://www.ros.org/wiki/xacro">
   <xacro:arg name="tf_prefix" default="" />
-  <xacro:include filename="$(find dynaarm_end_effectors)/urdf/weight_5kg.urdf.xacro" />
+  <xacro:include filename="$(find duatic_dynaarm_end_effectors)/urdf/freedrive_handle.urdf.xacro" />
   <link name="base_link" />
-  <!-- Add platform to base_link -->
-  <xacro:weight_5kg tf_prefix="$(arg tf_prefix)"
+  <!-- Add platform to world -->
+  <xacro:freedrive_handle tf_prefix="$(arg tf_prefix)"
               parent="base_link">
     <origin xyz="0 0 0.0" rpy="0 0 0" />
-  </xacro:weight_5kg>
+  </xacro:freedrive_handle>
 </robot>

File: duatic_dynaarm_end_effectors/urdf/hook.urdf.xacro (robot description, xacro)
@@ -21,16 +21,16 @@
 THE USE OF THIS SOFTWARE, EVEN IF ADVISED OF THE POSSIBILITY OF SUCH DAMAGE.
 -->
-<robot name="shovel_gripper_left" xmlns:xacro="http://www.ros.org/wiki/xacro">
+<robot name="hook" xmlns:xacro="http://www.ros.org/wiki/xacro">
   <!-- Link Definition -->
-<xacro:macro name="shovel_gripper_left" params="tf_prefix parent *origin">
-  <link name="${tf_prefix}shovel_link">
+<xacro:macro name="hook" params="tf_prefix parent *origin">
+  <link name="${tf_prefix}hook_link">
     <!-- Inertial Properties -->
     <inertial>
-      <origin xyz="0.006776 0.016062 0.062373" rpy="0 0 0"/>
-      <mass value="0.540"/>
+      <origin xyz="0.004832 -0.001237 0.033429" rpy="0 0 0"/>
+      <mass value="0.157"/>
       <inertia
-        ixx="0.001724034" ixy="-0.000233095"  ixz="-0.000205439"
-        iyy="0.001391918" iyz="0.000135485"
-        izz="0.001304677"/>
+        ixx="0.001677" ixy="0.0"  ixz="-0.000509"
+        iyy="0.001510" iyz="0.0"
+        izz="0.001501"/>
     </inertial>
     <!-- Visual -->
@@ -38,21 +38,18 @@
       <origin xyz="0 0 0" rpy="0 0 0"/>
       <geometry>
-      <mesh filename="file://$(find dynaarm_end_effectors)/meshes/shovel_gripper_left_mesh.stl" scale="1 1 1"/>
+      <mesh filename="file://$(find duatic_dynaarm_end_effectors)/meshes/hook.dae" scale="1 1 1"/>
       </geometry>
-      <material name="gray">
-        <color rgba="0.6 0.6 0.6 1.0"/>
-      </material>
     </visual>
     <collision>
       <origin xyz="0 0 0" rpy="0 0 0"/>
       <geometry>
-      <mesh filename="file://$(find dynaarm_end_effectors)/meshes/shovel_gripper_left_mesh.stl" scale="1 1 1"/>
+      <mesh filename="file://$(find duatic_dynaarm_end_effectors)/meshes/hook.dae" scale="1 1 1"/>
       </geometry>
     </collision>
   </link>
   <!-- Fixed Joint to parent link -->
-  <joint name="${tf_prefix}shovel_joint" type="fixed">
+  <joint name="${tf_prefix}hook_joint" type="fixed">
     <parent link="${parent}"/>
-    <child link="${tf_prefix}shovel_link"/>
+    <child link="${tf_prefix}hook_link"/>
     <xacro:insert_block name="origin" />
   </joint>

File: duatic_dynaarm_end_effectors/urdf/hook_standalone.urdf.xacro (robot description, xacro)
@@ -1,5 +1,5 @@
 <robot name="hook_on_world" xmlns:xacro="http://www.ros.org/wiki/xacro">
   <xacro:arg name="tf_prefix" default="" />
-  <xacro:include filename="$(find dynaarm_end_effectors)/urdf/hook.urdf.xacro" />
+  <xacro:include filename="$(find duatic_dynaarm_end_effectors)/urdf/hook.urdf.xacro" />
   <link name="base_link" />
   <!-- Add platform to world -->

File: duatic_dynaarm_end_effectors/urdf/shovel.urdf.xacro (robot description, xacro)
@@ -21,16 +21,16 @@
 THE USE OF THIS SOFTWARE, EVEN IF ADVISED OF THE POSSIBILITY OF SUCH DAMAGE.
 -->
-<robot name="freedrive_handle" xmlns:xacro="http://www.ros.org/wiki/xacro">
+<robot name="shovel" xmlns:xacro="http://www.ros.org/wiki/xacro">
   <!-- Link Definition -->
-<xacro:macro name="freedrive_handle" params="tf_prefix parent *origin">
-  <link name="${tf_prefix}freedrive_handle_link">
+<xacro:macro name="shovel" params="tf_prefix parent *origin">
+  <link name="${tf_prefix}shovel_link">
     <!-- Inertial Properties -->
     <inertial>
-      <origin xyz="0.0423 0 0" rpy="0 0 0"/>
-      <mass value="0.149"/>
+      <origin xyz="0.004832 -0.001237 0.033429" rpy="0 0 0"/>
+      <mass value="0.551"/>
       <inertia
-        ixx=" 0.0000520" ixy="0.0"  ixz="0.0"
-        iyy="0.0001585" iyz="0.0"
-        izz="0.0001585"/>
+        ixx="0.001677" ixy="0.0"  ixz="-0.000509"
+        iyy="0.001510" iyz="0.0"
+        izz="0.001501"/>
     </inertial>
     <!-- Visual -->
@@ -38,5 +38,5 @@
       <origin xyz="0 0 0" rpy="0 0 0"/>
       <geometry>
-      <mesh filename="file://$(find dynaarm_end_effectors)/meshes/freedrive_handle_mesh.stl" scale="1 1 1"/>
+      <mesh filename="file://$(find duatic_dynaarm_end_effectors)/meshes/shovel_mesh.stl" scale="1 1 1"/>
       </geometry>
       <material name="gray">
@@ -47,12 +47,12 @@
       <origin xyz="0 0 0" rpy="0 0 0"/>
       <geometry>
-      <mesh filename="file://$(find dynaarm_end_effectors)/meshes/freedrive_handle_mesh.stl" scale="1 1 1"/>
+      <mesh filename="file://$(find duatic_dynaarm_end_effectors)/meshes/shovel_mesh.stl" scale="1 1 1"/>
       </geometry>
     </collision>
   </link>
   <!-- Fixed Joint to parent link -->
-  <joint name="${tf_prefix}freedrive_handle_joint" type="fixed">
+  <joint name="${tf_prefix}shovel_joint" type="fixed">
     <parent link="${parent}"/>
-    <child link="${tf_prefix}freedrive_handle_link"/>
+    <child link="${tf_prefix}shovel_link"/>
     <xacro:insert_block name="origin" />
   </joint>

File: duatic_dynaarm_end_effectors/urdf/shovel_gripper_left.urdf.xacro (robot description, xacro)
@@ -21,16 +21,16 @@
 THE USE OF THIS SOFTWARE, EVEN IF ADVISED OF THE POSSIBILITY OF SUCH DAMAGE.
 -->
-<robot name="shovel_gripper_right" xmlns:xacro="http://www.ros.org/wiki/xacro">
+<robot name="shovel_gripper_left" xmlns:xacro="http://www.ros.org/wiki/xacro">
   <!-- Link Definition -->
-<xacro:macro name="shovel_gripper_right" params="tf_prefix parent *origin">
+<xacro:macro name="shovel_gripper_left" params="tf_prefix parent *origin">
   <link name="${tf_prefix}shovel_link">
     <!-- Inertial Properties -->
     <inertial>
-      <origin xyz="0.007887 -0.015220 0.059359" rpy="0 0 0"/>
-      <mass value="0.580724"/>
+      <origin xyz="0.006776 0.016062 0.062373" rpy="0 0 0"/>
+      <mass value="0.540"/>
       <inertia
-        ixx="0.001822" ixy="0.000232"  ixz="-0.000205"
-        iyy="0.001508" iyz="-0.000158"
-        izz="0.001357"/>
+        ixx="0.001724034" ixy="-0.000233095"  ixz="-0.000205439"
+        iyy="0.001391918" iyz="0.000135485"
+        izz="0.001304677"/>
     </inertial>
     <!-- Visual -->
@@ -38,5 +38,5 @@
       <origin xyz="0 0 0" rpy="0 0 0"/>
       <geometry>
-      <mesh filename="file://$(find dynaarm_end_effectors)/meshes/shovel_gripper_right_mesh.stl" scale="1 1 1"/>
+      <mesh filename="file://$(find duatic_dynaarm_end_effectors)/meshes/shovel_gripper_left_mesh.stl" scale="1 1 1"/>
       </geometry>
       <material name="gray">
@@ -47,5 +47,5 @@
       <origin xyz="0 0 0" rpy="0 0 0"/>
       <geometry>
-      <mesh filename="file://$(find dynaarm_end_effectors)/meshes/shovel_gripper_right_mesh.stl" scale="1 1 1"/>
+      <mesh filename="file://$(find duatic_dynaarm_end_effectors)/meshes/shovel_gripper_left_mesh.stl" scale="1 1 1"/>
       </geometry>
     </collision>

File: duatic_dynaarm_end_effectors/urdf/shovel_gripper_right.urdf.xacro (robot description, xacro)
@@ -21,16 +21,16 @@
 THE USE OF THIS SOFTWARE, EVEN IF ADVISED OF THE POSSIBILITY OF SUCH DAMAGE.
 -->
-<robot name="shovel" xmlns:xacro="http://www.ros.org/wiki/xacro">
+<robot name="shovel_gripper_right" xmlns:xacro="http://www.ros.org/wiki/xacro">
   <!-- Link Definition -->
-<xacro:macro name="shovel" params="tf_prefix parent *origin">
+<xacro:macro name="shovel_gripper_right" params="tf_prefix parent *origin">
   <link name="${tf_prefix}shovel_link">
     <!-- Inertial Properties -->
     <inertial>
-      <origin xyz="0.004832 -0.001237 0.033429" rpy="0 0 0"/>
-      <mass value="0.551"/>
+      <origin xyz="0.007887 -0.015220 0.059359" rpy="0 0 0"/>
+      <mass value="0.580724"/>
       <inertia
-        ixx="0.001677" ixy="0.0"  ixz="-0.000509"
-        iyy="0.001510" iyz="0.0"
-        izz="0.001501"/>
+        ixx="0.001822" ixy="0.000232"  ixz="-0.000205"
+        iyy="0.001508" iyz="-0.000158"
+        izz="0.001357"/>
     </inertial>
     <!-- Visual -->
@@ -38,5 +38,5 @@
       <origin xyz="0 0 0" rpy="0 0 0"/>
       <geometry>
-      <mesh filename="file://$(find dynaarm_end_effectors)/meshes/shovel_mesh.stl" scale="1 1 1"/>
+      <mesh filename="file://$(find duatic_dynaarm_end_effectors)/meshes/shovel_gripper_right_mesh.stl" scale="1 1 1"/>
       </geometry>
       <material name="gray">
@@ -47,5 +47,5 @@
       <origin xyz="0 0 0" rpy="0 0 0"/>
       <geometry>
-      <mesh filename="file://$(find dynaarm_end_effectors)/meshes/shovel_mesh.stl" scale="1 1 1"/>
+      <mesh filename="file://$(find duatic_dynaarm_end_effectors)/meshes/shovel_gripper_right_mesh.stl" scale="1 1 1"/>
       </geometry>
     </collision>

File: duatic_dynaarm_end_effectors/urdf/shovel_gripper_standalone.urdf.xacro (robot description, xacro)
@@ -1,6 +1,6 @@
 <robot name="shovel_on_world" xmlns:xacro="http://www.ros.org/wiki/xacro">
   <xacro:arg name="tf_prefix" default="" />
-  <xacro:include filename="$(find dynaarm_end_effectors)/urdf/shovel_gripper_right.urdf.xacro" />
-  <xacro:include filename="$(find dynaarm_end_effectors)/urdf/shovel_gripper_left.urdf.xacro" />
+  <xacro:include filename="$(find duatic_dynaarm_end_effectors)/urdf/shovel_gripper_right.urdf.xacro" />
+  <xacro:include filename="$(find duatic_dynaarm_end_effectors)/urdf/shovel_gripper_left.urdf.xacro" />
   <link name="base_link" />
   <!-- Add platform to base_link -->

File: duatic_dynaarm_end_effectors/urdf/shovel_standalone.urdf.xacro (robot description, xacro)
@@ -1,5 +1,5 @@
 <robot name="shovel_on_world" xmlns:xacro="http://www.ros.org/wiki/xacro">
   <xacro:arg name="tf_prefix" default="" />
-  <xacro:include filename="$(find dynaarm_end_effectors)/urdf/shovel.urdf.xacro" />
+  <xacro:include filename="$(find duatic_dynaarm_end_effectors)/urdf/shovel.urdf.xacro" />
   <link name="base_link" />
   <!-- Add platform to base_link -->

File: duatic_dynaarm_end_effectors/urdf/weight_5kg.urdf.xacro (robot description, xacro)
@@ -21,16 +21,16 @@
 THE USE OF THIS SOFTWARE, EVEN IF ADVISED OF THE POSSIBILITY OF SUCH DAMAGE.
 -->
-<robot name="hook" xmlns:xacro="http://www.ros.org/wiki/xacro">
+<robot name="weight_5kg" xmlns:xacro="http://www.ros.org/wiki/xacro">
   <!-- Link Definition -->
-<xacro:macro name="hook" params="tf_prefix parent *origin">
-  <link name="${tf_prefix}hook_link">
+<xacro:macro name="weight_5kg" params="tf_prefix parent *origin">
+  <link name="${tf_prefix}weight_5kg_link">
     <!-- Inertial Properties -->
     <inertial>
-      <origin xyz="0.004832 -0.001237 0.033429" rpy="0 0 0"/>
-      <mass value="0.157"/>
+      <origin xyz="0.026295 0 0.000104" rpy="0 0 0"/>
+      <mass value="5.417999"/>
       <inertia
-        ixx="0.001677" ixy="0.0"  ixz="-0.000509"
-        iyy="0.001510" iyz="0.0"
-        izz="0.001501"/>
+        ixx="0.031114" ixy="0.0"  ixz="0.000015"
+        iyy="0.015956" iyz="0.0"
+        izz=" 0.019591"/>
     </inertial>
     <!-- Visual -->
@@ -38,18 +38,21 @@
       <origin xyz="0 0 0" rpy="0 0 0"/>
       <geometry>
-      <mesh filename="file://$(find dynaarm_end_effectors)/meshes/hook.dae" scale="1 1 1"/>
+      <mesh filename="file://$(find duatic_dynaarm_end_effectors)/meshes/weight_mesh.stl" scale="1 1 1"/>
       </geometry>
+      <material name="gray">
+        <color rgba="0.6 0.6 0.6 1.0"/>
+      </material>
     </visual>
     <collision>
       <origin xyz="0 0 0" rpy="0 0 0"/>
       <geometry>
-      <mesh filename="file://$(find dynaarm_end_effectors)/meshes/hook.dae" scale="1 1 1"/>
+      <mesh filename="file://$(find duatic_dynaarm_end_effectors)/meshes/weight_mesh.stl" scale="1 1 1"/>
       </geometry>
     </collision>
   </link>
   <!-- Fixed Joint to parent link -->
-  <joint name="${tf_prefix}hook_joint" type="fixed">
+  <joint name="${tf_prefix}weight_5kg_joint" type="fixed">
     <parent link="${parent}"/>
-    <child link="${tf_prefix}hook_link"/>
+    <child link="${tf_prefix}weight_5kg_link"/>
     <xacro:insert_block name="origin" />
   </joint>

File: duatic_dynaarm_end_effectors/urdf/weight_5kg_standalone.urdf.xacro (robot description, xacro)
@@ -1,10 +1,10 @@
 <robot name="weight_on_world" xmlns:xacro="http://www.ros.org/wiki/xacro">
   <xacro:arg name="tf_prefix" default="" />
-  <xacro:include filename="$(find dynaarm_end_effectors)/urdf/freedrive_handle.urdf.xacro" />
+  <xacro:include filename="$(find duatic_dynaarm_end_effectors)/urdf/weight_5kg.urdf.xacro" />
   <link name="base_link" />
-  <!-- Add platform to world -->
-  <xacro:freedrive_handle tf_prefix="$(arg tf_prefix)"
+  <!-- Add platform to base_link -->
+  <xacro:weight_5kg tf_prefix="$(arg tf_prefix)"
               parent="base_link">
     <origin xyz="0 0 0.0" rpy="0 0 0" />
-  </xacro:freedrive_handle>
+  </xacro:weight_5kg>
 </robot>
