Commit message: Fixed the sim launch as default should be gazebo and not isaac.

File: duatic_dynaarm_single_example/duatic_dynaarm_single_example_description/urdf/dynaarm_single_example.urdf.xacro (robot description, xacro)
@@ -24,5 +24,5 @@
   <xacro:arg name="namespace" default="dynaarm1" />
   <xacro:include filename="$(find duatic_dynaarm_driver)/urdf/dynaarm.urdf.xacro" />
-  <link name="base_link" />
+<link name="base_link" />
   <link name="table">
     <visual>
@@ -41,8 +41,14 @@
       </geometry>
     </collision>
+    <inertial>
+      <mass value="10.0"/>
+      <origin xyz="0 0 0"/>
+      <inertia ixx="1.0" ixy="0.0" ixz="0.0" iyy="1.0" iyz="0.0" izz="1.0"/>
+    </inertial>
   </link>
   <joint name="table_joint" type="fixed">
     <parent link="base_link"/>
     <child link="table"/>
+    <origin xyz="0 0 -0.025" rpy="0 0 0"/>
   </joint>
   <!-- create an instance of the dynaarm and fix its base-->
@@ -57,8 +63,8 @@
     <origin xyz="0 0 0" rpy="0.0 0.0 0.0" />
   </xacro:dynaarm>
-  <!-- Gazebo Ros2 Control -->
+  <!-- Include the control plugin -->
   <xacro:include filename="$(find duatic_control)/urdf/plugins.urdf.xacro" />
   <xacro:control namespace="$(arg namespace)">
-    <remapping>cmd_vel:=cmd_vel</remapping> <!-- TODO: This line only exists, because otherwise the xacro doesn't compile -->
+    <remapping>cmd_vel:=/cmd_vel</remapping> <!-- TODO: This line only exists, because otherwise the xacro doesn't compile -->
   </xacro:control>
 </robot>
